Commit message: added camera feed, made the cameras lighter and not like bricks

File: spherical_robot_control/urdf/spherical_robot.urdf (robot description, URDF)
Before this commit: robot spherical_robot, 8 links, 7 joints
Links:
- added link camera_left_link
- added link camera_left_optical_frame
- added link camera_right_link
- added link camera_right_optical_frame
Joints:
- added joint camera_left_joint: type fixed, parent frame, child camera_left_link, origin xyz=0.19 0.21 0.0 rpy=0 0 0.0872665
- added joint camera_left_optical_joint: type fixed, parent camera_left_link, child camera_left_optical_frame, origin xyz=0 0 0 rpy=-1.5708 0 -1.5708
- added joint camera_right_joint: type fixed, parent frame, child camera_right_link, origin xyz=0.19 -0.21 0.0 rpy=0 0 -0.0872665
- added joint camera_right_optical_joint: type fixed, parent camera_right_link, child camera_right_optical_frame, origin xyz=0 0 0 rpy=-1.5708 0 -1.5708

Commit message: added a new inertial wheel for yaw control, i'm afraid of it but let's see what happens

File: spherical_robot_control/urdf/spherical_robot.urdf (robot description, URDF)
Before this commit: robot spherical_robot, 12 links, 11 joints
Links:
- removed link rw_w_link
- removed link rw_x_link
- removed link rw_y_link
- removed link rw_z_link
- added link rw_back_link
- added link rw_front_link
- added link rw_left_link
- added link rw_right_link
- added link rw_yaw_link
Joints:
- removed joint rw_w
- removed joint rw_x
- removed joint rw_y
- removed joint rw_z
- added joint rw_back: type continuous, parent frame, child rw_back_link, axis 0 0 1
- added joint rw_front: type continuous, parent frame, child rw_front_link, axis 0 0 1
- added joint rw_left: type continuous, parent frame, child rw_left_link, axis 0 0 1
- added joint rw_right: type continuous, parent frame, child rw_right_link, axis 0 0 1
- added joint rw_yaw: type continuous, parent frame, child rw_yaw_link, axis 0 0 1
- joint camera_left_joint: origin xyz=0.19 0.21 0.0 rpy=0 0 0.0872665 -> xyz=0.19 -0.21 0.0 rpy=3.14159 0 -0.0872665
- joint camera_right_joint: origin xyz=0.19 -0.21 0.0 rpy=0 0 -0.0872665 -> xyz=0.19 0.21 0.0 rpy=3.14159 0 0.0872665

Commit message: trying self collision and also simplifications to the robot, this would make it easier to modelize its dynamics

File: spherical_robot_control/urdf/spherical_robot.urdf (robot description, URDF)
Before this commit: robot spherical_robot, 12 links, 11 joints
Links:
- removed link motor_joint_1_link
- removed link motor_joint_2_link
Joints:
- removed joint motor_joint_1
- removed joint motor_joint_2
